Commit message: remove useless part of urdf

File: ur5_description/urdf/ur5_hitbot_with_ilc_platform.xacro.urdf (robot description, URDF)
Before this commit: robot ur5_hitbot_with_ilc_platform, 40 links, 39 joints
Links:
- removed link beam_support_robot_top
- removed link hitbot_base
- removed link hitbot_finger0
- removed link hitbot_finger0_tip
- removed link hitbot_finger1
- removed link hitbot_finger1_tip
- removed link hitbot_mask
- removed link tool0
- link operation_surface: geometry collision box size=0.7 0.6 0.025; visual box size=0.7 1.14 0.025
Joints:
- removed joint hitbot_base_finger0_joint
- removed joint hitbot_base_finger1_joint
- removed joint hitbot_base_mask_joint
- removed joint hitbot_finger0_tip_joint
- removed joint hitbot_finger1_tip_joint
- removed joint platform_base_beam_support_robot_top_joint
- removed joint tool0_hitbot_joint
- removed joint wrist_3_link-tool0_fixed_joint
- joint platform_base_robot_install_plate_joint: origin xyz=0.0                   0.0                   0.0825 rpy=0.0 0.0 0.0 -> xyz=0.05                   -0.2                   0.0 rpy=0.0 0.0 0.0; parent beam_support_robot_top -> operation_surface
