Commit message: update ur5 description

File: ur5_description/urdf/ur5_hitbot_with_ilc_platform.urdf.xacro (robot description, xacro)
@@ -20,5 +20,5 @@
   <xacro:include filename="$(find handson_description)/urdf/ilc_platform.urdf.xacro" />
   <!-- arm -->
-  <xacro:ur5_robot prefix="" joint_limited="false"/>
+  <!-- <xacro:ur5_robot prefix="" joint_limited="false"/> -->
   <!-- hand -->
   <xacro:include filename="$(find handson_description)/urdf/hitbot/hitbot.urdf.xacro" />

File: ur5_description/urdf/ur5_hitbot_with_ilc_platform.xacro.urdf (robot description, URDF)
Before this commit: robot ur5_hitbot_with_ilc_platform, 32 links, 31 joints
Links:
- added link camera_link; visual mesh filename=package://ur5_description/meshes/d435.dae
Joints:
- added joint camera_link: type fixed, parent wrist_3_link, child camera_link, origin xyz=0.0 0.0 0.0 ${pi/4} rpy=0.0 0.0 0.0
