Commit message: update description of ur5

File: ur5_description/ur5_with_realsense.xacro.urdf (robot description, URDF)
Before this commit: robot ur5_hitbot_with_ilc_platform, 33 links, 32 joints
Links:
- added link sucker_link; visual mesh filename=package://ur5_description/meshes/sucker.stl scale=0.0018 0.0018 0.0018
Joints:
- removed joint camera_link
- added joint camera_joint: type fixed, parent wrist_3_link, child camera_link, origin xyz=-0.07 0.08 0.0 rpy=-1.57 1.57 0.0
- added joint sucker_joint: type fixed, parent wrist_3_link, child sucker_link, origin xyz=0.0 0.0 0.0 rpy=0.0 0.0 3.14

File: ur5_description/urdf/ur5_with_realsense.xacro.urdf (robot description, URDF)
Before this commit: robot ur5_hitbot_with_ilc_platform, 34 links, 33 joints
Links:
- link sucker_link: geometry visual mesh filename=package://ur5_description/meshes/sucker.stl scale=0.0018 0.0018 0.0018
Joints:
- joint camera_joint: origin xyz=0.07 0.08 0.0 rpy=-1.57 1.57 0.0 -> xyz=-0.07 0.08 0.0 rpy=-1.57 1.57 0.0
- joint sucker_joint: origin xyz=0.0 0.1 0.0 rpy=0.0 0.0 0.0 -> xyz=0.0 0.0 0.0 rpy=0.0 0.0 3.14
